File: I2C-LEDStripDriver.brd (EAGLE design)
At the start: 109.9 x 100 mm, 31 parts, among them Q1 IRF540N, Q2 IRF540N, Q3 IRF540N, Q4 IRF540N, Q5 IRF540N, Q6 IRF540N, Q7 IRF540N, Q8 IRF540N, U1 PCA9685PW

Commit message: 2.0
Parts:
- removed A0: (no value), SPCoast:1X03
- removed C8: 150uF, SPCoast:0810-CAP
- removed I2C-1, I2C-2: CONNECTOR-I2CLEFT, SPCoast:I2C-L
- removed U$5: MOUNTINGHOLE, SPCoast:MOUNTINGHOLE
- added A6: (no value), SPCoast:1X03
- added C2: 0.1uF, SPCoast:0805-CAP
- added C3: 10uF, SPCoast:0805-CAP
- added C5: 150uF, SPCoast:0810-CAP
- added CON5, CON6: (no value), SPCoast:MSTBA2
- added R1, R10, R2, R3, R4, R5, R6, R7, R8, R9: 10k, SPCoast:0603-RES
- added U$1: MOUNTINGHOLE, SPCoast:MOUNTINGHOLE
- added U2: WemosD1, SPCoast:WEMOS-D1
- added VR1: 7805, SPCoast:TO-252
- CON1, CON2: value (none) -> GROVE-4P-2.0; device SPCoast:MSTBA4 -> SPCoast:4P-2.0
- CON3, CON4: device SPCoast:MSTBA2 -> SPCoast:MSTBA4
- Q1, Q2, Q3, Q4, Q5, Q6, Q7, Q8: value IRF540N -> DMN4468
- moved U$3 104.1 mm to (5.08, 85.1)
- moved U$2 91.9 mm to (95.2, 15.2)
- moved CON1 90.6 mm to (95.2, 26.7), turned to 270 degrees
- moved C1 70.0 mm to (9.14, 20.4), turned to 90 degrees
- moved CON2 62.7 mm to (95.2, 40.6), turned to 90 degrees
- moved C4 58.2 mm to (66.7, 59.1), turned to 270 degrees
- moved CON3 43.2 mm to (17.8, 73.7)
- moved CON4 34.3 mm to (41.9, 73.7)
- moved A1 24.1 mm to (21.6, 29.2)
- moved A2 19.1 mm to (24.1, 29.2)
- moved OSHW1 17.8 mm to (5.21, 15.2)
- moved U1 14.0 mm to (15.2, 20.3)
- moved A3 14.0 mm to (26.7, 29.2)
- moved A4 8.89 mm to (29.2, 29.2)
- moved POWER 6.48 mm to (82.5, 21.6)
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Connections:
- removed net B_DRIVE3: CON3.2, Q7.5, Q7.6, Q7.7, Q7.8
- removed net G_DRIVE3: CON4.2, Q8.5, Q8.6, Q8.7, Q8.8
- removed net VCCIO: A0.3, A1.3, A2.3, A3.3, A4.3, A5.3, C4.1, I2C-1.V+, I2C-1.V+@1, I2C-2.V+, I2C-2.V+@1, U1.28
- new net +3V3: A1.3, A2.3, A3.3, A4.3, A5.3, A6.3, C1.1, R1.2, R2.2, U1.28, U2.3V3
- new net +5V: C3.1, CON1.3, U2.5V, VR1.3
- new net W_DRIVE1: CON5.2, Q7.5, Q7.6, Q7.7, Q7.8
- new net W_DRIVE2: CON6.2, Q8.5, Q8.6, Q8.7, Q8.8
- net +12V: now also C2.1, C4.1, C5.+, CON2.3, CON2.4, CON5.1, CON6.1, VR1.1; no longer C1.1, C8.+, CON1.1, CON2.1
- net A0: now also A6.2; no longer A0.2
- net A1: now also A5.2; no longer A1.2
- net A2: now also A4.2; no longer A2.2
- net A4: now also A2.2; no longer A4.2
- net A5: now also A1.2; no longer A5.2
- net BLED1: now also R4.2
- net BLED2: now also R6.2
- net B_DRIVE1: now also CON3.4; no longer CON1.4
- net B_DRIVE2: now also CON4.4; no longer CON2.4
- net GLED1: now also R3.2
- net GLED2: now also R8.2
- net GND: now also A6.1, C2.2, C3.2, C5.-, CON1.4, CON2.1, CON2.2, R10.1, R3.1, R4.1, R5.1, R6.1, R7.1, R8.1, R9.1, U2.GND, VR1.2; no longer A0.1, C8.-, I2C-1.GND, I2C-1.GND@1, I2C-2.GND, I2C-2.GND@1
- net G_DRIVE1: now also CON3.3; no longer CON1.3
- net G_DRIVE2: now also CON4.3; no longer CON2.3
- net RLED1: now also R5.2
- net RLED2: now also R7.2
- net R_DRIVE1: now also CON3.2; no longer CON1.2
- net R_DRIVE2: now also CON4.2; no longer CON2.2
- net SCL: now also CON1.1, R2.1, U2.D3; no longer I2C-1.SCL, I2C-1.SCL@1, I2C-2.SCL, I2C-2.SCL@1
- net SDA: now also CON1.2, R1.1, U2.D2; no longer I2C-1.SDA, I2C-1.SDA@1, I2C-2.SDA, I2C-2.SDA@1
- net WLED1: now also R9.2
- net WLED2: now also R10.2
Routing:
- net VCCIO: track 169.6 -> 0.00 mm
- net GND: track 275.7 -> 155.7 mm
- net +3V3: track 0.00 -> 113.2 mm, vias 0 -> 2
- net +5V: track 0.00 -> 74.7 mm, vias 0 -> 1
- net +12V: track 0.00 -> 68.0 mm, vias 0 -> 1
- net SDA: track 114.7 -> 93.7 mm, vias 2 -> 1
- net GLED1: track 44.6 -> 64.1 mm
- net GLED2: track 50.9 -> 70.4 mm
- net SCL: track 110.7 -> 97.5 mm, vias 2 -> 0
- net BLED2: track 48.1 -> 60.5 mm
- net WLED2: track 80.1 -> 92.0 mm
- net W_DRIVE1: track 0.00 -> 9.50 mm
- net B_DRIVE3: track 9.50 -> 0.00 mm
- net W_DRIVE2: track 0.00 -> 9.50 mm
- net G_DRIVE3: track 9.50 -> 0.00 mm
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- added copper zone on layer 16, net +12V
- removed copper zone on layer 1, net +12V
Other:
- board text added: "+12v VIN"
- board text added: "+5v"
- board text added: "GND"
- board text added: "I2C"
- board text added: "I2C WiFi LED Strip Driver"
- board text added: "SCL"
- board text added: "SDA"
- board text added: "V2.0"
- board text removed: "I2C LED Strip Driver"
- board text removed: "V1.0"

Commit message: default address (0) and silkscreen updates
Parts:
- added CON7: GROVE-4P-2.0, SPCoast:4P-2.0
- moved OSHW1 58.2 mm to (52.2, 49.5)
Connections:
- net +3V3: now also R1.1, R2.1; no longer R1.2, R2.2
- net +5V: now also CON7.3
- net GND: now also CON7.4
- net SCL: now also CON7.1, R2.2; no longer R2.1
- net SDA: now also CON7.2, R1.2; no longer R1.1
Routing:
- net GND: track 155.7 -> 207.4 mm
- net +5V: track 74.7 -> 87.8 mm
- net SCL: track 97.5 -> 95.2 mm, vias 0 -> 1
- net +3V3: track 113.2 -> 114.7 mm
- net SDA: track 93.7 -> 94.9 mm, vias 1 -> 0
Other:
- board text added: "+12v VIN To Expanders"
- board text added: "2019.03 2020.07"
- board text added: "Go Bears!"
- board text added: "I2C LED Strip Driver"
- board text added: "Power for LEDS"
- board text added: "V2.0b"
- board text removed: "+12v VIN"
- board text removed: "2019.03"
- board text removed: "I2C WiFi LED Strip Driver"
- board text removed: "V2.0"
