File: I2C-LEDStripDriver.sch (EAGLE design)
At the start: 31 parts, among them Q1 IRF540N, Q2 IRF540N, Q3 IRF540N, Q4 IRF540N, Q5 IRF540N, Q6 IRF540N, Q7 IRF540N, Q8 IRF540N, U1 PCA9685PW

Commit message: 2.0
Parts:
- removed A0: (no value), SPCoast:JUMPER-3PTH-LOCK
- removed C8: 150uF, SPCoast:CAP-POL0810
- removed I2C-1, I2C-2: CONNECTOR-I2CLEFT, SPCoast:CONNECTOR-I2CLEFT
- removed U$5: MOUNTINGHOLE, SPCoast:MOUNTINGHOLE
- added A6: (no value), SPCoast:JUMPER-3PTH-LOCK
- added C2: 0.1uF, SPCoast:CAP0805
- added C3: 10uF, SPCoast:CAP0805
- added C5: 150uF, SPCoast:CAP-POL0810
- added CON5, CON6: (no value), SPCoast:CONNECTOR-M02MSTBA2
- added R1, R10, R2, R3, R4, R5, R6, R7, R8, R9: 10k, SPCoast:R0603-RES
- added U$1: MOUNTINGHOLE, SPCoast:MOUNTINGHOLE
- added U2: WemosD1, SPCoast:WEMOS-D1V1
- added VR1: 7805, SPCoast:VREG-DPAK-5
- CON1, CON2: value (none) -> GROVE-4P-2.0; device SPCoast:CONNECTOR-M045.08 -> SPCoast:CONNECTOR-GROVE-4P-2.0-3470130P1
- CON3, CON4: device SPCoast:CONNECTOR-M02MSTBA2 -> SPCoast:CONNECTOR-M045.08
- Q1, Q2, Q3, Q4, Q5, Q6, Q7, Q8: value IRF540N -> DMN4468
Connections:
- removed net B_DRIVE3: CON3.B, Q7.D
- removed net G_DRIVE3: CON4.B, Q8.D
- removed net VCCIO: A0.3, A1.3, A2.3, A3.3, A4.3, A5.3, C4.1, I2C-1.V+, I2C-2.V+, U1.VDD
- new net +3V3: A1.3, A2.3, A3.3, A4.3, A5.3, A6.3, C1.1, R1.2, R2.2, U1.VDD, U2.3V3
- new net +5V: C3.1, CON1.3, U2.5V, VR1.OUT
- new net W_DRIVE1: CON5.B, Q7.D
- new net W_DRIVE2: CON6.B, Q8.D
- net +12V: now also C2.1, C4.1, C5.+, CON2.3, CON2.4, CON3.1, CON4.1, CON5.A, CON6.A, VR1.IN; no longer C1.1, C8.+, CON1.1, CON2.1, CON3.A, CON4.A
- net A0: now also A6.2; no longer A0.2
- net A1: now also A5.2; no longer A1.2
- net A2: now also A4.2; no longer A2.2
- net A4: now also A2.2; no longer A4.2
- net A5: now also A1.2; no longer A5.2
- net BLED1: now also R4.2
- net BLED2: now also R6.2
- net B_DRIVE1: now also CON3.4; no longer CON1.4
- net B_DRIVE2: now also CON4.4; no longer CON2.4
- net GLED1: now also R3.2
- net GLED2: now also R8.2
- net GND: now also A6.1, C2.2, C3.2, C5.-, CON1.4, CON2.1, CON2.2, R10.1, R3.1, R4.1, R5.1, R6.1, R7.1, R8.1, R9.1, U2.GND, VR1.GND; no longer A0.1, C8.-, I2C-1.GND, I2C-2.GND
- net G_DRIVE1: now also CON3.3; no longer CON1.3
- net G_DRIVE2: now also CON4.3; no longer CON2.3
- net RLED1: now also R5.2
- net RLED2: now also R7.2
- net R_DRIVE1: now also CON3.2; no longer CON1.2
- net R_DRIVE2: now also CON4.2; no longer CON2.2
- net SCL: now also CON1.1, R2.1, U2.D3; no longer I2C-1.SCL, I2C-2.SCL
- net SDA: now also CON1.2, R1.1, U2.D2; no longer I2C-1.SDA, I2C-2.SDA
- net WLED1: now also R9.2
- net WLED2: now also R10.2
Other:
- note added: "2.0"
- note removed: "1.0"
- moved on the sheet: A1, A2, A3, A4, A5, C1, C4, POWER, Q1, Q2, Q3, Q4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

Commit message: default address (0) and silkscreen updates
Parts:
- added CON7: GROVE-4P-2.0, SPCoast:CONNECTOR-GROVE-4P-2.0-3470130P1
Connections:
- net +3V3: now also R1.1, R2.1; no longer R1.2, R2.2
- net +5V: now also CON7.3
- net GND: now also CON7.4
- net SCL: now also CON7.1, R2.2; no longer R2.1
- net SDA: now also CON7.2, R1.2; no longer R1.1
Other:
- note added: "/* * Dest, Src, V1, W1, W2, R1, G1, B1, R2, G2, B2 */ #define W2 0 #define W1 1 #define R2 3 #define G2 2 #define B2 4 #define R1 6 #define G1 5 #define B1 7 // Index from ADC maps to Control Packet order which maps to LED driver order... static byte color_channel_map[8] = { W1, B1, G1, R1, W2, B2, G2, R2 };"
- note added: "2.0b"
- note added: "Drives 2x RGB strips and 2x White strips with a 12v/15A power supply (For backdrop and valence controlled lighting) v2.0b: default address=0, silkscreen changes"
- note removed: "2.0"
- note removed: "Drives 2x RGB strips and 2x White strips with a 12v/15A power supply (For backdrop and valence controlled lighting)"
- moved on the sheet: C1, U1
